File: kicad/drummodul/Final_Platine_1/KiKAD_Final_Platine_1_V1.kicad_sch (KiCad schematic)
At the start: 45 parts, among them J1 Conn_02x08_Odd_Even, J4 Conn_01x03_Pin, Q1 Q_NPN_ECB, Q2 Q_NPN_ECB, Q3 Q_NPN_ECB, U1 NE555P, U2 AD8603

Commit message: Platinen sind Ready
Parts:
- J4: footprint (none) -> Connector_JST:JST_EH_S3B-EH_1x03_P2.50mm_Horizontal
- Microcontroller_Input1: renamed from Microcontroller_Input; footprint (none) -> Connector_JST:JST_EH_S2B-EH_1x02_P2.50mm_Horizontal
- Output1: renamed from Output; footprint (none) -> Connector_JST:JST_EH_S2B-EH_1x02_P2.50mm_Horizontal
- RV2: footprint (none) -> Connector_JST:JST_XH_B3B-XH-A_1x03_P2.50mm_Vertical
Connections:
- net at C12.1, R19.2: now also U2.3 (+)
Changed lines of the file:
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@@
   (junction (at 132.08 149.86) (diameter 0) (color 0 0 0 0)
+  )
+  (junction (at 249.682 102.87) (diameter 0) (color 0 0 0 0)
   )
   (no_connect (at 22.86 139.7))
@@
     (stroke (width 0) (type default))
   )
+  (wire (pts (xy 249.682 102.87) (xy 252.73 102.87))
+    (stroke (width 0) (type default))
+  )
   (wire (pts (xy 204.47 149.86) (xy 204.47 146.05))
     (stroke (width 0) (type default))
@@
       (effects (font (size 1.27 1.27)))
     )
-    (property "Footprint" "" (at 267.716 109.982 0)
+    (property "Footprint" "Connector_JST:JST_XH_B3B-XH-A_1x03_P2.50mm_Vertical" (at 267.716 109.982 0)
       (effects (font (size 1.27 1.27)) hide)
     )
@@
       (effects (font (size 1.27 1.27)))
     )
-    (property "Footprint" "" (at 52.832 53.594 0)
+    (property "Footprint" "Connector_JST:JST_EH_S3B-EH_1x03_P2.50mm_Horizontal" (at 52.832 53.594 0)
       (effects (font (size 1.27 1.27)) hide)
     )
@@
   (symbol (lib_id "Connector:Conn_01x02_Pin") (at 13.97 50.8 0) (unit 1)
     (in_bom yes) (on_board yes) (dnp no)
-    (property "Reference" "Microcontroller_Input" (at 22.86 42.545 0)
+    (property "Reference" "Microcontroller_Input1" (at 22.86 42.545 0)
       (effects (font (size 1.27 1.27)))
     )
@@
       (effects (font (size 1.27 1.27)))
     )
-    (property "Footprint" "" (at 13.97 50.8 0)
+    (property "Footprint" "Connector_JST:JST_EH_S2B-EH_1x02_P2.50mm_Horizontal" (at 13.97 50.8 0)
       (effects (font (size 1.27 1.27)) hide)
     )
@@
       (project "KiKAD_Final_Platine_1_V1"
         (path "/06aebb48-3bd9-4517-ad22-b5366be0f5d8"
-          (reference "Microcontroller_Input") (unit 1)
+          (reference "Microcontroller_Input1") (unit 1)
         )
       )
@@
   (symbol (lib_id "Connector:Conn_01x02_Pin") (at 280.67 107.95 180) (unit 1)
     (in_bom yes) (on_board yes) (dnp no)
-    (property "Reference" "Output" (at 279.527 102.743 0)
+    (property "Reference" "Output1" (at 279.527 102.743 0)
       (effects (font (size 1.27 1.27)))
     )
@@
       (effects (font (size 1.27 1.27)))
     )
-    (property "Footprint" "" (at 280.67 107.95 0)
+    (property "Footprint" "Connector_JST:JST_EH_S2B-EH_1x02_P2.50mm_Horizontal" (at 280.67 107.95 0)
       (effects (font (size 1.27 1.27)) hide)
     )
@@
       (project "KiKAD_Final_Platine_1_V1"
         (path "/06aebb48-3bd9-4517-ad22-b5366be0f5d8"
-          (reference "Output") (unit 1)
-        )
-      )
+          (reference "Output1") (unit 1)
+        )
+      )
