File: kicad/drummodul/Final_Platine_2/KiKAD_Final_Platine_2_V1.kicad_sch (KiCad schematic)
At the start: 33 parts, among them J1 Conn_02x08_Odd_Even, J4 Conn_01x03_Pin, Q1 Q_NPN_ECB, Q2 Q_NPN_ECB, U1 NE555P, U2 AD8603

Commit message: Platinen sind Ready
Parts:
- J4, RV2: footprint (none) -> Connector_JST:JST_EH_S3B-EH_1x03_P2.50mm_Horizontal
- L1: footprint (none) -> Inductor_SMD:L_1206_3216Metric_Pad1.42x1.75mm_HandSolder
- MicrontrollerInput1: renamed from MicrontrollerInput; footprint (none) -> Connector_JST:JST_EH_S2B-EH_1x02_P2.50mm_Horizontal
- Noise_Input1: renamed from Noise_Input; footprint (none) -> Connector_JST:JST_EH_S2B-EH_1x02_P2.50mm_Horizontal
- Output1: renamed from Output; footprint (none) -> Connector_JST:JST_EH_S2B-EH_1x02_P2.50mm_Horizontal
