File: kicad/drummodul/Final_Platine_Noise/KiKAD_Final_Platine_Noise_V1.kicad_sch (KiCad schematic)
At the start: 10 parts, among them J1 Conn_02x08_Odd_Even, Q2 Q_NPN_ECB, U2 AD8603

Commit message: Platinen sind Ready
Parts:
- Output1: renamed from Output; footprint (none) -> Connector_JST:JST_EH_S2B-EH_1x02_P2.50mm_Horizontal
Changed lines of the file:
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@@
   (symbol (lib_id "Connector:Conn_01x02_Pin") (at 138.176 128.016 180) (unit 1)
     (in_bom yes) (on_board yes) (dnp no)
-    (property "Reference" "Output" (at 136.398 121.158 0)
+    (property "Reference" "Output1" (at 136.398 121.158 0)
       (effects (font (size 1.27 1.27)) (justify right))
     )
@@
       (effects (font (size 1.27 1.27)) (justify right))
     )
-    (property "Footprint" "" (at 138.176 128.016 0)
+    (property "Footprint" "Connector_JST:JST_EH_S2B-EH_1x02_P2.50mm_Horizontal" (at 138.176 128.016 0)
       (effects (font (size 1.27 1.27)) hide)
     )
@@
       (project "KiKAD_Final_Platine_Noise_V1"
         (path "/06aebb48-3bd9-4517-ad22-b5366be0f5d8"
-          (reference "Output") (unit 1)
+          (reference "Output1") (unit 1)
         )
       )
