File: kicad/Finale Platine/KiKAD_Endplatine_V1.kicad_sch (KiCad schematic)
At the start: 58 parts, among them J1 Conn_02x08_Odd_Even, J4 Conn_01x03_Pin, Q1 Q_NPN_ECB, Q2 Q_NPN_ECB, Q3 Q_NPN_ECB, Q4 Q_NPN_ECB, U1 NE555P, U2 TL074, U3 TL074, U5 TL074

Commit message: alles mögliche
Connections:
- net at C14.1, R27.2: now also Q4.1 (E); no longer Q4.2 (C)
Changed lines of the file:
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@@
   (junction (at 71.628 50.546) (diameter 0) (color 0 0 0 0)
-  )
-  (junction (at 109.22 93.472) (diameter 0) (color 0 0 0 0)
   )
   (junction (at 164.084 102.362) (diameter 0) (color 0 0 0 0)
@@
     (stroke (width 0) (type default))
   )
-  (wire (pts (xy 109.22 92.71) (xy 109.22 93.472))
-    (stroke (width 0) (type default))
-  )
   (wire (pts (xy 122.4788 96.8756) (xy 116.6368 96.8756))
     (stroke (width 0) (type default))
@@
     (stroke (width 0) (type default))
   )
-  (wire (pts (xy 161.798 91.948) (xy 164.084 91.948))
-    (stroke (width 0) (type default))
-  )
   (wire (pts (xy 63.5 59.69) (xy 61.468 59.69))
     (stroke (width 0) (type default))
   )
-  (wire (pts (xy 109.22 93.472) (xy 161.798 93.472))
-    (stroke (width 0) (type default))
-  )
   (wire (pts (xy 109.22 134.62) (xy 109.22 149.86))
     (stroke (width 0) (type default))
@@
     (stroke (width 0) (type default))
   )
-  (wire (pts (xy 161.798 93.472) (xy 161.798 91.948))
-    (stroke (width 0) (type default))
-  )
   (wire (pts (xy 109.22 111.4552) (xy 116.6368 111.4552))
     (stroke (width 0) (type default))
@@
     (stroke (width 0) (type default))
   )
-  (wire (pts (xy 109.22 93.472) (xy 109.22 96.8756))
+  (wire (pts (xy 109.22 92.71) (xy 109.22 96.8756))
     (stroke (width 0) (type default))
   )
@@
     )
   )
-  (symbol (lib_id "Device:Q_NPN_ECB") (at 145.288 45.974 0) (unit 1)
-    (in_bom yes) (on_board yes) (dnp no) (fields_autoplaced)
-    (property "Reference" "Q4" (at 151.13 45.339 0)
+  (symbol (lib_id "Device:Q_NPN_ECB") (at 145.288 45.974 0) (mirror x) (unit 1)
+    (in_bom yes) (on_board yes) (dnp no)
+    (property "Reference" "Q4" (at 151.13 46.609 0)
       (effects (font (size 1.27 1.27)) (justify left))
     )
-    (property "Value" "Q_NPN_ECB" (at 151.13 47.879 0)
+    (property "Value" "Q_NPN_ECB" (at 151.13 44.069 0)
       (effects (font (size 1.27 1.27)) (justify left))
     )
-    (property "Footprint" "Package_TO_SOT_SMD:SOT-23-3" (at 150.368 43.434 0)
+    (property "Footprint" "Package_TO_SOT_SMD:SOT-23-3" (at 150.368 48.514 0)
       (effects (font (size 1.27 1.27)) hide)
     )
@@
         )
       )
+    )
+  )
+  (symbol (lib_id "power:+12V") (at 164.084 91.948 0) (unit 1)
+    (in_bom yes) (on_board yes) (dnp no) (fields_autoplaced)
+    (property "Reference" "#PWR02" (at 164.084 95.758 0)
+      (effects (font (size 1.27 1.27)) hide)
+    )
+    (property "Value" "+12V" (at 164.084 88.138 0)
+      (effects (font (size 1.27 1.27)))
+    )
+    (property "Footprint" "" (at 164.084 91.948 0)
+      (effects (font (size 1.27 1.27)) hide)
+    )
+    (property "Datasheet" "" (at 164.084 91.948 0)
+      (effects (font (size 1.27 1.27)) hide)
+    )
+    (pin "1")
+    (instances
+      (project "KiKAD_Endplatine_V1"
+        (path "/06aebb48-3bd9-4517-ad22-b5366be0f5d8"
+          (reference "#PWR02") (unit 1)
+        )
+      )
