File: kicad/Finale Platine/KiKAD_Endplatine_V2.kicad_sch (KiCad schematic)
At the start: 68 parts, among them J1 Conn_02x08_Odd_Even, J4 Conn_01x03_Pin, Q1 Q_NPN_ECB, Q2 Q_NPN_ECB, Q3/+1/+1 Q_NPN_ECB, U1 NE555P, U2 TL074

Commit message: kleines Platinenupdate
Parts:
- C1: value C -> 1u
Connections:
- net GND: now also +/R17.2, R12.2
- net at C16.2: now also Output1.2 (Pin_2), R12.1; no longer R12.2
- net at +/C15.2: now also +/+1.2, +/R17.1, C4/C2/C2.1, C7/+/+1.1, R9/+/+1.1; no longer +/R17.2
Other:
- moved on the sheet: +/R17, R12
Changed lines of the file:
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@@
   (junction (at 116.84 86.868) (diameter 0) (color 0 0 0 0)
   )
+  (junction (at 233.172 40.386) (diameter 0) (color 0 0 0 0)
+  )
   (junction (at 54.356 37.338) (diameter 0) (color 0 0 0 0)
   )
@@
   )
   (junction (at 131.826 149.86) (diameter 0) (color 0 0 0 0)
+  )
+  (junction (at 246.38 108.966) (diameter 0) (color 0 0 0 0)
   )
   (junction (at 16.256 129.54) (diameter 0) (color 0 0 0 0)
@@
     (stroke (width 0) (type default))
   )
+  (wire (pts (xy 246.38 108.966) (xy 257.048 108.966))
+    (stroke (width 0) (type default))
+  )
   (wire (pts (xy 71.628 62.738) (xy 71.628 67.056))
     (stroke (width 0) (type default))
@@
     (stroke (width 0) (type default))
   )
+  (wire (pts (xy 233.172 40.386) (xy 237.744 40.386))
+    (stroke (width 0) (type default))
+  )
   (wire (pts (xy 109.22 86.868) (xy 109.22 99.06))
     (stroke (width 0) (type default))
@@
     (stroke (width 0) (type default))
   )
-  (wire (pts (xy 253.492 108.966) (xy 257.048 108.966))
-    (stroke (width 0) (type default))
-  )
   (wire (pts (xy 41.656 129.54) (xy 45.466 129.54))
     (stroke (width 0) (type default))
@@
     (stroke (width 0) (type default))
   )
-  (wire (pts (xy 244.094 108.966) (xy 245.872 108.966))
+  (wire (pts (xy 244.094 108.966) (xy 246.38 108.966))
     (stroke (width 0) (type default))
   )
@@
   )
   (wire (pts (xy 84.582 121.412) (xy 84.582 129.54))
+    (stroke (width 0) (type default))
+  )
+  (wire (pts (xy 230.124 40.386) (xy 233.172 40.386))
     (stroke (width 0) (type default))
   )
@@
   (symbol (lib_id "Device:C_Small") (at 241.554 108.966 90) (unit 1)
     (in_bom yes) (on_board yes) (dnp no)
-    (property "Reference" "C16" (at 243.586 112.268 90)
+    (property "Reference" "C16" (at 239.776 112.268 90)
       (effects (font (size 1.27 1.27)))
     )
@@
   (symbol (lib_id "Device:C_Small") (at 227.584 40.386 90) (unit 1)
     (in_bom yes) (on_board yes) (dnp no)
-    (property "Reference" "+/C15" (at 227.6856 43.4848 90)
+    (property "Reference" "+/C15" (at 227.076 35.306 90)
       (effects (font (size 1.27 1.27)))
     )
@@
   (symbol (lib_id "Device:C") (at 177.927 56.007 90) (unit 1)
     (in_bom yes) (on_board yes) (dnp no)
-    (property "Reference" "C1" (at 174.244 53.34 90)
-      (effects (font (size 1.27 1.27)))
-    )
-    (property "Value" "C" (at 177.927 52.316 90)
+    (property "Reference" "C1" (at 177.8 59.944 90)
+      (effects (font (size 1.27 1.27)))
+    )
+    (property "Value" "1u" (at 177.546 62.23 90)
       (effects (font (size 1.27 1.27)))
     )
@@
     )
   )
+  (symbol (lib_id "power:GND") (at 246.38 116.586 0) (unit 1)
+    (in_bom yes) (on_board yes) (dnp no) (fields_autoplaced)
+    (property "Reference" "#PWR024" (at 246.38 122.936 0)
+      (effects (font (size 1.27 1.27)) hide)
+    )
+    (property "Value" "GND" (at 246.38 121.666 0)
+      (effects (font (size 1.27 1.27)))
+    )
+    (property "Footprint" "" (at 246.38 116.586 0)
+      (effects (font (size 1.27 1.27)) hide)
+    )
+    (property "Datasheet" "" (at 246.38 116.586 0)
+      (effects (font (size 1.27 1.27)) hide)
+    )
+    (pin "1")
+    (instances
+      (project "KiKAD_Endplatine_V2"
+        (path "/06aebb48-3bd9-4517-ad22-b5366be0f5d8"
+          (reference "#PWR024") (unit 1)
+        )
+      )
+    )
+  )
   (symbol (lib_id "Amplifier_Operational:TL074") (at 160.655 37.846 0) (unit 1)
     (in_bom yes) (on_board yes) (dnp no)
@@
     )
   )
-  (symbol (lib_id "Device:R") (at 233.934 40.386 270) (unit 1)
-    (in_bom yes) (on_board yes) (dnp no)
-    (property "Reference" "+/R17" (at 233.934 37.084 90)
-      (effects (font (size 1.27 1.27)))
-    )
-    (property "Value" "1k" (at 233.934 42.926 90)
-      (effects (font (size 1.27 1.27)))
-    )
-    (property "Footprint" "Resistor_SMD:R_1206_3216Metric_Pad1.30x1.75mm_HandSolder" (at 233.934 38.608 90)
-      (effects (font (size 1.27 1.27)) hide)
-    )
-    (property "Datasheet" "~" (at 233.934 40.386 0)
+  (symbol (lib_id "Device:R") (at 233.172 44.196 0) (unit 1)
+    (in_bom yes) (on_board yes) (dnp no)
+    (property "Reference" "+/R17" (at 228.854 43.688 0)
+      (effects (font (size 1.27 1.27)))
+    )
+    (property "Value" "1k" (at 235.458 45.466 0)
+      (effects (font (size 1.27 1.27)))
+    )
+    (property "Footprint" "Resistor_SMD:R_1206_3216Metric_Pad1.30x1.75mm_HandSolder" (at 231.394 44.196 90)
+      (effects (font (size 1.27 1.27)) hide)
+    )
+    (property "Datasheet" "~" (at 233.172 44.196 0)
       (effects (font (size 1.27 1.27)) hide)
     )
@@
     )
   )
-  (symbol (lib_id "Device:R") (at 249.682 108.966 270) (unit 1)
-    (in_bom yes) (on_board yes) (dnp no)
-    (property "Reference" "R12" (at 249.682 106.426 90)
-      (effects (font (size 1.27 1.27)))
-    )
-    (property "Value" "1k" (at 249.682 111.506 90)
-      (effects (font (size 1.27 1.27)))
-    )
-    (property "Footprint" "Resistor_SMD:R_1206_3216Metric_Pad1.30x1.75mm_HandSolder" (at 249.682 107.188 90)
-      (effects (font (size 1.27 1.27)) hide)
-    )
-    (property "Datasheet" "~" (at 249.682 108.966 0)
+  (symbol (lib_id "Device:R") (at 246.38 112.776 0) (unit 1)
+    (in_bom yes) (on_board yes) (dnp no)
+    (property "Reference" "R12" (at 249.936 112.522 0)
+      (effects (font (size 1.27 1.27)))
+    )
+    (property "Value" "1k" (at 248.92 114.808 0)
+      (effects (font (size 1.27 1.27)))
+    )
+    (property "Footprint" "Resistor_SMD:R_1206_3216Metric_Pad1.30x1.75mm_HandSolder" (at 244.602 112.776 90)
+      (effects (font (size 1.27 1.27)) hide)
+    )
+    (property "Datasheet" "~" (at 246.38 112.776 0)
       (effects (font (size 1.27 1.27)) hide)
     )
@@
   (symbol (lib_id "Device:R_Potentiometer") (at 181.356 47.752 90) (unit 1)
     (in_bom yes) (on_board yes) (dnp no)
-    (property "Reference" "+/RV3" (at 183.134 51.054 90)
+    (property "Reference" "+/RV3" (at 184.15 51.562 90)
       (effects (font (size 1.27 1.27)))
     )
@@
         )
       )
+    )
+  )
+  (symbol (lib_id "power:GND") (at 233.172 48.006 0) (unit 1)
+    (in_bom yes) (on_board yes) (dnp no) (fields_autoplaced)
+    (property "Reference" "#PWR025" (at 233.172 54.356 0)
+      (effects (font (size 1.27 1.27)) hide)
+    )
+    (property "Value" "GND" (at 233.172 53.086 0)
+      (effects (font (size 1.27 1.27)))
+    )
+    (property "Footprint" "" (at 233.172 48.006 0)
+      (effects (font (size 1.27 1.27)) hide)
+    )
+    (property "Datasheet" "" (at 233.172 48.006 0)
+      (effects (font (size 1.27 1.27)) hide)
+    )
+    (pin "1")
+    (instances
+      (project "KiKAD_Endplatine_V2"
+        (path "/06aebb48-3bd9-4517-ad22-b5366be0f5d8"
+          (reference "#PWR025") (unit 1)
+        )
+      )
