File: kicad/Finale Platine/KiKAD_Endplatine_V2.kicad_sch (KiCad schematic)
At the start: 68 parts, among them J1 Conn_02x08_Odd_Even, J4 Conn_01x03_Pin, Q1 Q_NPN_ECB, Q2 Q_NPN_ECB, Q3/+1/+1 Q_NPN_ECB, U1 NE555P, U2 TL074

Commit message: jetzt hoffentlich
Parts:
- removed +/+1, -/-/-1: 1000k, Resistor_SMD:R_1206_3216Metric_Pad1.30x1.75mm_HandSolder, symbol Device:R
- removed +/Q4, Q1, Q2, Q3/+1/+1: Q_NPN_ECB, Package_TO_SOT_SMD:SOT-23-3, symbol Device:Q_NPN_ECB
- removed +/R1: 100k, Resistor_SMD:R_1206_3216Metric_Pad1.30x1.75mm_HandSolder, symbol Device:R
- removed +/RV2, +/RV3: 10k, Connector_JST:JST_EH_S3B-EH_1x03_P2.50mm_Horizontal, symbol Device:R_Potentiometer
- removed C1: C, Capacitor_SMD:C_1206_3216Metric_Pad1.33x1.80mm_HandSolder, symbol Device:C
- removed J4: Conn_01x03_Pin, Connector_JST:JST_EH_S3B-EH_1x03_P2.50mm_Horizontal, symbol Connector:Conn_01x03_Pin
- removed unit 3 of U2
- added Q1, Q2, Q3, Q4: Q_NPN_BEC, Package_TO_SOT_SMD:SOT-23-3, symbol Device:Q_NPN_BEC
- added Taster1: Conn_01x02_Pin, Connector_JST:JST_EH_B2B-EH-A_1x02_P2.50mm_Vertical, symbol Connector:Conn_01x02_Pin
- C31: renamed from C21; value 1p -> 100n
- C32: renamed from C22; value 100n -> 10n
- C33: renamed from C23; value 10p -> 10u
- D2: value C5/D2/D2 -> D2
- MicrontrollerInput1: footprint Connector_JST:JST_EH_S3B-EH_1x03_P2.50mm_Horizontal -> Connector_JST:JST_EH_B2B-EH-A_1x02_P2.50mm_Vertical
- Output1: footprint Connector_JST:JST_EH_S3B-EH_1x03_P2.50mm_Horizontal -> Connector_JST:JST_EH_S2B-EH_1x02_P2.50mm_Horizontal
- R32: value 10k -> 47k
- R33: value 214 -> 220
- R34: value 1k -> 10k
- RV1: renamed from RV/RV/+1; footprint Connector_JST:JST_EH_S3B-EH_1x03_P2.50mm_Horizontal -> Connector_JST:JST_EH_B2B-EH-A_1x02_P2.50mm_Vertical
- RV2: renamed from RV1k/-/-1; footprint Connector_JST:JST_EH_S3B-EH_1x03_P2.50mm_Horizontal -> Connector_JST:JST_EH_B2B-EH-A_1x02_P2.50mm_Vertical
- RV3: renamed from RV2; footprint Connector_JST:JST_EH_S3B-EH_1x03_P2.50mm_Horizontal -> Connector_JST:JST_EH_B2B-EH-A_1x02_P2.50mm_Vertical
- RV4: renamed from +/RV1; footprint Connector_JST:JST_EH_S3B-EH_1x03_P2.50mm_Horizontal -> Connector_JST:JST_EH_B2B-EH-A_1x02_P2.50mm_Vertical
- Trimpoti1: renamed from RV/+1; footprint Connector_JST:JST_EH_S3B-EH_1x03_P2.50mm_Horizontal -> Connector_JST:JST_EH_B3B-EH-A_1x03_P2.50mm_Vertical
- renumbered C3/C1 to C1, C16 to C10, C4/C2/C2 to C2, +/C14 to C21, +/C15 to C23, R9/+/+1 to C3, C24 to C34, C7/+/+1 to C4, C6/R1/C3 to C5, +/C6/C6 to C6, C8/C5/C5 to C7, C1/+/-1 to C8, C9/+/-1 to C9, +/D1 to D1, +/L1 to L1, +/L2/L2 to L2, +/L3 to L3, R1/R1/R1 to R1, R12/-1 to R10, R14/R4/R4 to R11, R2/R5/+1 to R12, R16/+1/R5 to R13, R4/+/-1 to R14, R3/+/+1 to R15, R17/+/+1 to R16, R6/+/+1 to R17, R10 to R18, R12 to R19, D1/R2/R2 to R2, +/R27 to R21, +/R28 to R22, +/R29 to R24, +/R30 to R25, +/R17 to R26, R8/1/+1 to R3, R7/-/-1 to R4, R11/+/+1 to R5, R10/-1 to R6, C6/R3 to R7
Connections:
- net GND: now also R19.2, R26.2, Q3.2 (E), Q4.1 (B), Taster1.2 (Pin_2)
- net at C4.2, C6.2, C7.1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: now also Q1.3 (C)
- net at C21.1, R21.2: now also Q4.2 (E)
- net at C10.2: now also Output1.2 (Pin_2), R19.1; no longer R19.2
- net at C32.1, R32.2: now also Q3.3 (C), Taster1.1 (Pin_1)
- net at R31.2: now also Q3.1 (B)
- net at R6.2, R7.1: now also C3.2, C5.1
- net at R24.1: now also U2.1, U2.2 (-)
- net at C23.2: now also C2.1, C3.1, C4.1, R26.1; no longer R26.2
- net at C9.1, R14.1, R15.2: now also Q2.3 (C)
- net at C8.2, R14.2: now also Q2.1 (B)
- net at D2.1 (K), R5.2, R6.1: now also Q1.1 (B)
- net at R16.2: now also Q2.2 (E)
- net at R10.2: now also Q1.2 (E)
- net at R3.2: now also RV1.1; no longer RV1.3
- no-connect marks 11 -> 9
Other:
- moved on the sheet: C21, C23, R19, R24, R25, R26, RV1, RV4, U2A, U2B
