File: kicad/Finale Platine/KiKAD_Endplatine_V2.kicad_pcb (KiCad board)
At the start: 2 copper layers, 100 x 80 mm, 70 parts, among them J1 Conn_02x08_Odd_Even, J4 Conn_01x03_Pin, Q1 Q_NPN_ECB, Q2 Q_NPN_ECB, Q3/+1/+1 Q_NPN_ECB, U1 NE555P, U2 TL074

Commit message: jetzt hoffentlich
Parts:
- removed +/+1, -/-/-1: 1000k, Resistor_SMD:R_1206_3216Metric_Pad1.30x1.75mm_HandSolder
- removed +/Q4, Q3/+1/+1: Q_NPN_ECB, Package_TO_SOT_SMD:SOT-23-3
- removed +/R1: 100k, Resistor_SMD:R_1206_3216Metric_Pad1.30x1.75mm_HandSolder
- removed +/RV2, +/RV3: 10k, Connector_JST:JST_EH_S3B-EH_1x03_P2.50mm_Horizontal
- removed J4: Conn_01x03_Pin, Connector_JST:JST_EH_S3B-EH_1x03_P2.50mm_Horizontal
- added Q3: Q_NPN_BEC, Package_TO_SOT_SMD:SOT-23-3, F.Cu at (185.0, 39.4)
- added Q4: Q_NPN_BEC, Package_TO_SOT_SMD:SOT-23-3, F.Cu at (166.5, 94.5)
- added Taster1: Conn_01x02_Pin, Connector_JST:JST_EH_B2B-EH-A_1x02_P2.50mm_Vertical, F.Cu at (181.2, 54.3)
- C31: renamed from C21; value 1p -> 100n
- C32: renamed from C22; value 100n -> 10n
- C33: renamed from C23; value 10p -> 10u
- D2: value C5/D2/D2 -> D2
- MicrontrollerInput1: footprint Connector_JST:JST_EH_S3B-EH_1x03_P2.50mm_Horizontal -> Connector_JST:JST_EH_B2B-EH-A_1x02_P2.50mm_Vertical
- Output1: footprint Connector_JST:JST_EH_S3B-EH_1x03_P2.50mm_Horizontal -> Connector_JST:JST_EH_S2B-EH_1x02_P2.50mm_Horizontal
- Q1, Q2: value Q_NPN_ECB -> Q_NPN_BEC
- R32: value 10k -> 47k
- R33: value 214 -> 220
- R34: value 1k -> 10k
- RV1: renamed from RV/RV/+1; footprint Connector_JST:JST_EH_S3B-EH_1x03_P2.50mm_Horizontal -> Connector_JST:JST_EH_B2B-EH-A_1x02_P2.50mm_Vertical
- RV2: renamed from RV1k/-/-1; footprint Connector_JST:JST_EH_S3B-EH_1x03_P2.50mm_Horizontal -> Connector_JST:JST_EH_B2B-EH-A_1x02_P2.50mm_Vertical
- RV3: renamed from RV2; footprint Connector_JST:JST_EH_S3B-EH_1x03_P2.50mm_Horizontal -> Connector_JST:JST_EH_B2B-EH-A_1x02_P2.50mm_Vertical
- RV4: renamed from +/RV1; footprint Connector_JST:JST_EH_S3B-EH_1x03_P2.50mm_Horizontal -> Connector_JST:JST_EH_B2B-EH-A_1x02_P2.50mm_Vertical
- Trimpoti1: renamed from RV/+1; footprint Connector_JST:JST_EH_S3B-EH_1x03_P2.50mm_Horizontal -> Connector_JST:JST_EH_B3B-EH-A_1x03_P2.50mm_Vertical
- moved Q2 64.0 mm to (133.5, 73.1), turned to 90 degrees
- moved R24 11.7 mm to (177.0, 90.0), turned to -90 degrees
- moved C10 11.5 mm to (194.0, 69.5), turned to 90 degrees
- moved RV1 4.50 mm to (123.5, 101.0), turned to 180 degrees
- moved C23 2.92 mm to (170.5, 106.5)
- moved Q1 0.71 mm to (136.0, 89.5), turned to 90 degrees
- moved C1 0.35 mm to (117.5, 111.5)
- renumbered C3/C1 to C1, C16 to C10, C4/C2/C2 to C2, +/C14 to C21, +/C15 to C23, R9/+/+1 to C3, C24 to C34, C7/+/+1 to C4, C6/R1/C3 to C5, +/C6/C6 to C6, C8/C5/C5 to C7, C1/+/-1 to C8, C9/+/-1 to C9, +/D1 to D1, +/L1 to L1, +/L2/L2 to L2, +/L3 to L3, R1/R1/R1 to R1, R12/-1 to R10, R14/R4/R4 to R11, R2/R5/+1 to R12, R16/+1/R5 to R13, R4/+/-1 to R14, R3/+/+1 to R15, R17/+/+1 to R16, R6/+/+1 to R17, R10 to R18, R12 to R19, D1/R2/R2 to R2, +/R27 to R21, +/R28 to R22, +/R29 to R24, +/R30 to R25, +/R17 to R26, R8/1/+1 to R3, R7/-/-1 to R4, R11/+/+1 to R5, R10/-1 to R6, C6/R3 to R7
Connections:
- C10 pad 1: Net-(C16-Pad1) -> Net-(C10-Pad1)
- C10 pad 2: Net-(C16-Pad2) -> Net-(Output1-Pin_2)
- C2 pad 1: Net-(+/+1-Pad2) -> Net-(C2-Pad1)
- C23 pad 1: Net-(+/C15-Pad1) -> Net-(C23-Pad1)
- C23 pad 2: Net-(+/C15-Pad2) -> Net-(C2-Pad1)
- C3 pad 1: Net-(+/+1-Pad2) -> Net-(C2-Pad1)
- C3 pad 2: Net-(-/-/-1-Pad2) -> Net-(C3-Pad2)
- C32 pad 1: Net-(J4-Pin_2) -> Net-(Q3-C)
- C4 pad 1: Net-(+/+1-Pad2) -> Net-(C2-Pad1)
- C5 pad 1: Net-(-/-/-1-Pad2) -> Net-(C3-Pad2)
- C8 pad 2: Net-(Q3/+1/+1-B) -> Net-(Q2-B)
- C9 pad 1: Net-(Q3/+1/+1-C) -> Net-(Q2-C)
- Q1 pad 1: Net-(Q1-E) -> Net-(D2-K)
- Q1 pad 2: Net-(Q1-C) -> Net-(Q1-E)
- Q1 pad 3: Net-(D2-K) -> Net-(Q1-C)
- Q2 pad 1: GND -> Net-(Q2-B)
- Q2 pad 2: Net-(J4-Pin_2) -> Net-(Q2-E)
- Q2 pad 3: Net-(Q2-B) -> Net-(Q2-C)
- R14 pad 1: Net-(Q3/+1/+1-C) -> Net-(Q2-C)
- R14 pad 2: Net-(Q3/+1/+1-B) -> Net-(Q2-B)
- R15 pad 2: Net-(Q3/+1/+1-C) -> Net-(Q2-C)
- R16 pad 2: Net-(Q3/+1/+1-E) -> Net-(Q2-E)
- R19 pad 2: Net-(C16-Pad2) -> GND
- R24 pad 1: Net-(+/R29-Pad1) -> Net-(U2A--)
- R25 pad 2: Net-(+/C15-Pad1) -> Net-(C23-Pad1)
- R26 pad 1: Net-(+/+1-Pad2) -> Net-(C2-Pad1)
- R26 pad 2: Net-(+/C15-Pad2) -> GND
- R3 pad 2: Net-(R8/1/+1-Pad2) -> Net-(R3-Pad2)
- R31 pad 2: Net-(Q2-B) -> Net-(Q3-B)
- R32 pad 2: Net-(J4-Pin_2) -> Net-(Q3-C)
- R6 pad 2: Net-(+/RV2-Pad2) -> Net-(C3-Pad2)
- R7 pad 1: Net-(+/RV2-Pad2) -> Net-(C3-Pad2)
- RV1 pad 1: unconnected-(RV/RV/+1-Pad1) -> Net-(R3-Pad2)
- RV3 pad 2: Net-(C16-Pad1) -> Net-(C10-Pad1)
Routing:
- net Net-(C2-Pad1): track 0.00 -> 125.7 mm
- net Net-(+/+1-Pad2): track 121.6 -> 0.00 mm
- net Net-(+/C15-Pad1): track 42.2 -> 0.00 mm
- net Net-(+/RV2-Pad2): track 39.2 -> 0.00 mm
- net Net-(+/R29-Pad1): track 52.2 -> 18.8 mm
- net Net-(C3-Pad2): track 0.00 -> 30.5 mm
- net Net-(C16-Pad1): track 23.0 -> 0.00 mm
- net Net-(Q3/+1/+1-C): track 21.4 -> 0.00 mm
- net Net-(Q2-C): track 0.00 -> 21.4 mm
- net Net-(-/-/-1-Pad2): track 21.1 -> 0.00 mm
- net Net-(J4-Pin_2): track 17.0 -> 0.00 mm
- net Net-(U2A--): track 13.3 -> 29.8 mm
- net Net-(Q3-C): track 0.00 -> 15.9 mm
- net Net-(+/C15-Pad2): track 14.3 -> 0.00 mm
- net Net-(Q3/+1/+1-B): track 13.4 -> 0.00 mm
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