File: kicad/Finale Platine/KiKAD_Endplatine_V2-backups/KiKAD_Endplatine_V2-2023-09-11_175844/KiKAD_Endplatine_V1.kicad_sch (KiCad schematic)
At the start: 68 parts, among them J1 Conn_02x08_Odd_Even, J4 Conn_01x03_Pin, Q1 Q_NPN_ECB, Q2 Q_NPN_ECB, Q3/+1/+1 Q_NPN_ECB, U1 NE555P, U2 TL074

Commit message: aufräumaktion
Parts:
- removed +/L1, +/L3: 100m, Inductor_THT:L_Radial_D12.0mm_P6.00mm_Murata_1900R, symbol Device:L
- removed +/R1: 100k, Resistor_SMD:R_1206_3216Metric_Pad1.30x1.75mm_HandSolder, symbol Device:R
- removed +/RV1, +/RV2, +/RV3, RV/+1, RV/RV/+1, RV1k/-/-1: 10k, Connector_JST:JST_EH_S3B-EH_1x03_P2.50mm_Horizontal, symbol Device:R_Potentiometer
- removed C1: C, Capacitor_SMD:C_1206_3216Metric_Pad1.33x1.80mm_HandSolder, symbol Device:C
- removed C6/R1/C3: 1000k, Resistor_SMD:R_1206_3216Metric_Pad1.30x1.75mm_HandSolder, symbol Device:R
- removed R12/-1: 100, Resistor_SMD:R_1206_3216Metric_Pad1.30x1.75mm_HandSolder, symbol Device:R
- removed unit 5 of U2
- removed unit 2 of U2
- removed unit 3 of U2
- removed unit 4 of U2
- added U3, U5: TL074, symbol Amplifier_Operational:TL074
- D2: value C5/D2/D2 -> D
- L2: renamed from +/L2/L2; value 100m -> 1m; footprint Inductor_THT:L_Radial_D12.0mm_P6.00mm_Murata_1900R -> Inductor_SMD:L_1206_3216Metric_Pad1.42x1.75mm_HandSolder
- MicrontrollerInput1, Output1: footprint Connector_JST:JST_EH_S3B-EH_1x03_P2.50mm_Horizontal -> Connector_JST:JST_EH_S2B-EH_1x02_P2.50mm_Horizontal
- U2: footprint Package_DIP:DIP-14_W7.62mm -> (none)
- renumbered C3/C1 to C1, C21 to C10, C7/+/+1 to C11, C1/+/-1 to C12, C9/+/-1 to C13, +/C14 to C14, +/C15 to C15, C4/C2/C2 to C2, R9/+/+1 to C3, C22 to C4, C8/C5/C5 to C5, +/C6/C6 to C6, C24 to C7, C23 to C8, +/D1 to D1, Q3/+1/+1 to Q3, +/Q4 to Q4, R1/R1/R1 to R1, R8/1/+1 to R14, R7/-/-1 to R15, -/-/-1 to R16, +/R17 to R17, R11/+/+1 to R19, D1/R2/R2 to R2, C6/R3 to R20, +/+1 to R21, R2/R5/+1 to R22, R16/+1/R5 to R23, R4/+/-1 to R24, R3/+/+1 to R25, R17/+/+1 to R26, +/R27 to R27, +/R28 to R28, +/R29 to R29, R10/-1 to R3, +/R30 to R30, R14/R4/R4 to R4, R31 to R6, R6/+/+1 to R7, R32 to R7, R33 to R8, R34 to R9
Connections:
- net +12V: now also L2.1
- net GND: now also C3.2, Q1.1 (E), R16.2, U3.3 (+); no longer R10.1
- net at R10.2, RV2.1: now also U2.2 (-)
- net at C16.1, RV2.2: now also U2.1
- net at RV2.3: now also R10.1
- net at L2.2: now also C11.2, C5.1, C6.2, Q1.2 (C), R19.1, R4.2
- net at C13.2, R7.2: now also U2.3 (+)
- net at R29.2: now also U5.1, U5.2 (-)
- net at R30.1: now also R29.1, U3.2 (-)
- net at R15.1, R2.2: now also R14.2
- net at C15.1, R30.2: now also U3.1
- net at C14.2, R28.1: now also U5.3 (+); no longer U2.3 (+)
- no-connect marks 11 -> 6
Other:
- moved on the sheet: C14, C16, C5, C6, L2, Output1, Q4, R10, R12, R14, R24, R27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
