File: kicad/Finale Platine/KiKAD_Endplatine_V2-backups/KiKAD_Endplatine_V2-2023-09-11_175844/KiKAD_Endplatine_V2.kicad_pcb (KiCad board)
At the start: 2 copper layers, 100 x 80 mm, 70 parts, among them J1 Conn_02x08_Odd_Even, J4 Conn_01x03_Pin, Q1 Q_NPN_ECB, Q2 Q_NPN_ECB, Q3/+1/+1 Q_NPN_ECB, U1 NE555P, U2 TL074

Commit message: neue beschriftung in KiCad
Parts:
- D2: value C5/D2/D2 -> D2
- J4, MicrontrollerInput1, Output1: footprint Connector_JST:JST_EH_S3B-EH_1x03_P2.50mm_Horizontal -> Connector_JST:JST_EH_S2B-EH_1x02_P2.50mm_Horizontal
- RV1: renamed from RV/RV/+1; footprint Connector_JST:JST_EH_S3B-EH_1x03_P2.50mm_Horizontal -> Connector_JST:JST_EH_S2B-EH_1x02_P2.50mm_Horizontal
- RV2: renamed from +/RV2; footprint Connector_JST:JST_EH_S3B-EH_1x03_P2.50mm_Horizontal -> Connector_JST:JST_EH_S2B-EH_1x02_P2.50mm_Horizontal
- RV3: renamed from RV1k/-/-1; footprint Connector_JST:JST_EH_S3B-EH_1x03_P2.50mm_Horizontal -> Connector_JST:JST_EH_S2B-EH_1x02_P2.50mm_Horizontal
- RV4: renamed from RV2; footprint Connector_JST:JST_EH_S3B-EH_1x03_P2.50mm_Horizontal -> Connector_JST:JST_EH_S2B-EH_1x02_P2.50mm_Horizontal
- RV5: renamed from +/RV3; footprint Connector_JST:JST_EH_S3B-EH_1x03_P2.50mm_Horizontal -> Connector_JST:JST_EH_S2B-EH_1x02_P2.50mm_Horizontal
- RV6: renamed from +/RV1; footprint Connector_JST:JST_EH_S3B-EH_1x03_P2.50mm_Horizontal -> Connector_JST:JST_EH_S2B-EH_1x02_P2.50mm_Horizontal
- moved RV3 3.78 mm to (149.2, 84.0)
- moved Q4 1.35 mm to (166.0, 94.0), turned to -90 degrees
- renumbered C3/C1 to C1, C4/C2/C2 to C2, +/C14 to C21, C1 to C22, +/C15 to C23, R9/+/+1 to C3, C21 to C31, C22 to C32, C23 to C33, C24 to C34, C7/+/+1 to C4, C6/R1/C3 to C5, +/C6/C6 to C6, C8/C5/C5 to C7, C1/+/-1 to C8, C9/+/-1 to C9, +/D1 to D1, +/L1 to L1, +/L2/L2 to L2, +/L3 to L3, Q3/+1/+1 to Q2, Q2 to Q3, +/Q4 to Q4, R1/R1/R1 to R1, R12/-1 to R10, R14/R4/R4 to R11, R2/R5/+1 to R12, R16/+1/R5 to R13, R4/+/-1 to R14, R3/+/+1 to R15, R17/+/+1 to R16, R6/+/+1 to R17, R10 to R18, R12 to R19, D1/R2/R2 to R2, +/R27 to R21, +/R28 to R22, +/R1 to R23, +/R29 to R24, +/R30 to R25, +/R17 to R26, R8/1/+1 to R3, R7/-/-1 to R4, R11/+/+1 to R5, R10/-1 to R6, C6/R3 to R7, -/-/-1 to R8, +/+1 to R9, RV/+1 to RV_Trim1
Connections:
- C16 pad 2: Net-(C16-Pad2) -> Net-(Output1-Pin_2)
- C2 pad 1: Net-(+/+1-Pad2) -> Net-(C2-Pad1)
- C21 pad 1: Net-(+/Q4-C) -> Net-(Q4-E)
- C23 pad 2: Net-(+/C15-Pad2) -> Net-(C2-Pad1)
- C3 pad 1: Net-(+/+1-Pad2) -> Net-(C2-Pad1)
- C4 pad 1: Net-(+/+1-Pad2) -> Net-(C2-Pad1)
- Q4 pad 1: unconnected-(+/Q4-E-Pad1) -> Net-(Q4-E)
- Q4 pad 2: Net-(+/Q4-C) -> unconnected-(Q4-C-Pad2)
- R10 pad 1: Net-(R12/-1-Pad1) -> Net-(R10-Pad1)
- R19 pad 2: Net-(C16-Pad2) -> GND
- R21 pad 2: Net-(+/Q4-C) -> Net-(Q4-E)
- R26 pad 1: Net-(+/+1-Pad2) -> Net-(C2-Pad1)
- R26 pad 2: Net-(+/C15-Pad2) -> GND
- R3 pad 2: Net-(R8/1/+1-Pad2) -> Net-(R3-Pad2)
- R9 pad 2: Net-(+/+1-Pad2) -> Net-(C2-Pad1)
- RV3 pad 1: Net-(R12/-1-Pad1) -> GND
- RV3 pad 2: GND -> Net-(R10-Pad1)
Routing:
- net Net-(C2-Pad1): track 0.00 -> 125.1 mm
- net Net-(+/+1-Pad2): track 121.6 -> 0.00 mm
- net Net-(+/C15-Pad2): track 14.3 -> 0.00 mm
- net Net-(R10-Pad1): track 0.00 -> 9.85 mm
- net Net-(+/Q4-C): track 8.14 -> 0.00 mm
- net Net-(Q4-E): track 0.00 -> 7.53 mm
- net +12V: track 264.0 -> 270.4 mm
- net Net-(R8/1/+1-Pad2): track 5.72 -> 0.00 mm
- net Net-(R3-Pad2): track 0.00 -> 5.72 mm
- net Net-(R12/-1-Pad1): track 5.20 -> 0.00 mm
- net Net-(Output1-Pin_2): track 11.7 -> 16.1 mm
- net Net-(C16-Pad2): track 2.96 -> 0.00 mm
- net GND: vias 8 -> 11

Commit message: Anfang von Bautteilliste
Parts:
- renumbered C16 to C10, J4 to Taster1
Changed lines of the file:
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@@
   (net 3 "Net-(C2-Pad1)")
   (net 4 "Net-(D2-A)")
-  (net 5 "Net-(J4-Pin_2)")
+  (net 5 "Net-(Q3-C)")
   (net 6 "Net-(U1-TR)")
   (net 7 "Net-(Q1-C)")
@@
   (net 16 "Net-(Q4-E)")
   (net 17 "Net-(C22-Pad2)")
-  (net 18 "Net-(C16-Pad1)")
+  (net 18 "Net-(C10-Pad1)")
   (net 19 "Net-(C23-Pad1)")
   (net 20 "Net-(D1-A)")
@@
   (net 25 "unconnected-(J1-Pin_14-Pad14)")
   (net 26 "unconnected-(J1-Pin_16-Pad16)")
-  (net 27 "unconnected-(J4-Pin_1-Pad1)")
+  (net 27 "unconnected-(Taster1-Pin_1-Pad1)")
   (net 28 "Net-(MicrontrollerInput1-Pin_1)")
   (net 29 "Net-(Output1-Pin_2)")
@@
       (net 2 "GND") (pinfunction "E") (pintype "passive"))
     (pad "2" smd roundrect (at -1.1375 0.95) (size 1.325 0.6) (layers "F.Cu" "F.Paste" "F.Mask") (roundrect_rratio 0.25)
-      (net 5 "Net-(J4-Pin_2)") (pinfunction "C") (pintype "passive"))
+      (net 5 "Net-(Q3-C)") (pinfunction "C") (pintype "passive"))
     (pad "3" smd roundrect (at 1.1375 0) (size 1.325 0.6) (layers "F.Cu" "F.Paste" "F.Mask") (roundrect_rratio 0.25)
       (net 41 "Net-(Q3-B)") (pinfunction "B") (pintype "passive"))
@@
       (stroke (width 0.1) (type solid)) (layer "F.Fab"))
     (pad "1" smd roundrect (at -1.5625 0 180) (size 1.325 1.8) (layers "F.Cu" "F.Paste" "F.Mask") (roundrect_rratio 0.1886792453)
-      (net 5 "Net-(J4-Pin_2)") (pintype "passive"))
+      (net 5 "Net-(Q3-C)") (pintype "passive"))
     (pad "2" smd roundrect (at 1.5625 0 180) (size 1.325 1.8) (layers "F.Cu" "F.Paste" "F.Mask") (roundrect_rratio 0.1886792453)
       (net 6 "Net-(U1-TR)") (pintype "passive"))
@@
       (net 6 "Net-(U1-TR)") (pintype "passive"))
     (pad "2" smd roundrect (at 1.55 0) (size 1.3 1.75) (layers "F.Cu" "F.Paste" "F.Mask") (roundrect_rratio 0.1923076923)
-      (net 5 "Net-(J4-Pin_2)") (pintype "passive"))
+      (net 5 "Net-(Q3-C)") (pintype "passive"))
     (model "${KICAD6_3DMODEL_DIR}/Resistor_SMD.3dshapes/R_1206_3216Metric.wrl"
       (offset (xyz 0 0 0))
@@
       (net 39 "Net-(U2D--)") (pinfunction "1") (pintype "passive"))
     (pad "2" thru_hole oval (at 2.5 0 90) (size 1.7 2) (drill 1) (layers "*.Cu" "*.Mask")
-      (net 18 "Net-(C16-Pad1)") (pinfunction "2") (pintype "passive"))
+      (net 18 "Net-(C10-Pad1)") (pinfunction "2") (pintype "passive"))
     (model "${KICAD6_3DMODEL_DIR}/Connector_JST.3dshapes/JST_EH_S2B-EH_1x02_P2.50mm_Horizontal.wrl"
       (offset (xyz 0 0 0))
@@
       (net 39 "Net-(U2D--)") (pinfunction "-") (pintype "input"))
     (pad "14" thru_hole oval (at 7.62 0) (size 1.6 1.6) (drill 0.8) (layers "*.Cu" "*.Mask")
-      (net 18 "Net-(C16-Pad1)") (pintype "output"))
+      (net 18 "Net-(C10-Pad1)") (pintype "output"))
     (model "${KICAD6_3DMODEL_DIR}/Package_DIP.3dshapes/DIP-14_W7.62mm.wrl"
       (offset (xyz 0 0 0))
@@
     (property "ki_keywords" "connector")
     (attr through_hole)
-    (fp_text reference "J4" (at 1.25 -7.9 180) (layer "F.SilkS")
+    (fp_text reference "Taster1" (at 1.25 -7.9 180) (layer "F.SilkS")
         (effects (font (size 1 1) (thickness 0.15)))
     )
@@
       (stroke (width 0.1) (type solid)) (layer "F.Fab"))
     (pad "1" thru_hole roundrect (at 0 0 180) (size 1.7 2) (drill 1) (layers "*.Cu" "*.Mask") (roundrect_rratio 0.147059)
-      (net 27 "unconnected-(J4-Pin_1-Pad1)") (pinfunction "Pin_1") (pintype "passive+no_connect"))
+      (net 27 "unconnected-(Taster1-Pin_1-Pad1)") (pinfunction "Pin_1") (pintype "passive+no_connect"))
     (pad "2" thru_hole oval (at 2.5 0 180) (size 1.7 2) (drill 1) (layers "*.Cu" "*.Mask")
-      (net 5 "Net-(J4-Pin_2)") (pinfunction "Pin_2") (pintype "passive"))
+      (net 5 "Net-(Q3-C)") (pinfunction "Pin_2") (pintype "passive"))
     (model "${KICAD6_3DMODEL_DIR}/Connector_JST.3dshapes/JST_EH_S2B-EH_1x02_P2.50mm_Horizontal.wrl"
       (offset (xyz 0 0 0))
@@
     (property "ki_keywords" "capacitor cap")
     (attr smd)
-    (fp_text reference "C16" (at 0 -1.85) (layer "F.SilkS")
+    (fp_text reference "C10" (at 0 -1.85) (layer "F.SilkS")
         (effects (font (size 1 1) (thickness 0.15)))
     )
@@
       (stroke (width 0.1) (type solid)) (layer "F.Fab"))
     (pad "1" smd roundrect (at -1.5625 0) (size 1.325 1.8) (layers "F.Cu" "F.Paste" "F.Mask") (roundrect_rratio 0.1886792453)
-      (net 18 "Net-(C16-Pad1)") (pintype "passive"))
+      (net 18 "Net-(C10-Pad1)") (pintype "passive"))
     (pad "2" smd roundrect (at 1.5625 0) (size 1.325 1.8) (layers "F.Cu" "F.Paste" "F.Mask") (roundrect_rratio 0.1886792453)
       (net 29 "Net-(Output1-Pin_2)") (pintype "passive"))

Commit message: Bautteilliste Update
Neue Bautteilliste jtzt in Doku Ordner
KiCad Namensstruktur verändert und jaaa
Parts:
- removed R8, R9: 1000k, Resistor_SMD:R_1206_3216Metric_Pad1.30x1.75mm_HandSolder
- removed RV2: 10k, Connector_JST:JST_EH_S2B-EH_1x02_P2.50mm_Horizontal
- C31: value 1p -> 100n
- C32: value 100n -> 10n
- C33: value 10p -> 10u
- R32: value 10k -> 47k
- R33: value 214 -> 220
- R34: value 1k -> 10k
- RV3: value 10k -> 1k
- moved R7 3.33 mm to (155.5, 105.5)
- moved RV1 1.60 mm to (120.2, 102.0)
- moved C10 0.06 mm to (182.9, 66.0)
Connections:
- R6 pad 2: Net-(R6-Pad2) -> Net-(C3-Pad2)
- R7 pad 1: Net-(R6-Pad2) -> Net-(C3-Pad2)
- RV1 pad 1: unconnected-(RV1-Pad1) -> Net-(R2-Pad2)
- RV1 pad 2: Net-(R2-Pad2) -> Net-(R3-Pad2)
Routing:
- net Net-(R6-Pad2): track 38.8 -> 0.00 mm
- net Net-(C2-Pad1): track 125.1 -> 98.6 mm
- net Net-(C3-Pad2): track 21.1 -> 27.8 mm
- net Net-(U2D-+): track 141.4 -> 142.7 mm
