File: kicad/Finale Platine/KiKAD_Endplatine_V2-backups/KiKAD_Endplatine_V2-2023-09-11_175844/KiKAD_Endplatine_V2.kicad_sch (KiCad schematic)
At the start: 68 parts, among them J1 Conn_02x08_Odd_Even, J4 Conn_01x03_Pin, Q1 Q_NPN_ECB, Q2 Q_NPN_ECB, Q3/+1/+1 Q_NPN_ECB, U1 NE555P, U2 TL074

Commit message: neue beschriftung in KiCad
Parts:
- D2: value C5/D2/D2 -> D2
- J4, MicrontrollerInput1, Output1: footprint Connector_JST:JST_EH_S3B-EH_1x03_P2.50mm_Horizontal -> Connector_JST:JST_EH_S2B-EH_1x02_P2.50mm_Horizontal
- RV1: renamed from RV/RV/+1; footprint Connector_JST:JST_EH_S3B-EH_1x03_P2.50mm_Horizontal -> Connector_JST:JST_EH_S2B-EH_1x02_P2.50mm_Horizontal
- RV2: renamed from +/RV2; footprint Connector_JST:JST_EH_S3B-EH_1x03_P2.50mm_Horizontal -> Connector_JST:JST_EH_S2B-EH_1x02_P2.50mm_Horizontal
- RV3: renamed from RV1k/-/-1; footprint Connector_JST:JST_EH_S3B-EH_1x03_P2.50mm_Horizontal -> Connector_JST:JST_EH_S2B-EH_1x02_P2.50mm_Horizontal
- RV4: renamed from RV2; footprint Connector_JST:JST_EH_S3B-EH_1x03_P2.50mm_Horizontal -> Connector_JST:JST_EH_S2B-EH_1x02_P2.50mm_Horizontal
- RV5: renamed from +/RV3; footprint Connector_JST:JST_EH_S3B-EH_1x03_P2.50mm_Horizontal -> Connector_JST:JST_EH_S2B-EH_1x02_P2.50mm_Horizontal
- RV6: renamed from +/RV1; footprint Connector_JST:JST_EH_S3B-EH_1x03_P2.50mm_Horizontal -> Connector_JST:JST_EH_S2B-EH_1x02_P2.50mm_Horizontal
- renumbered C3/C1 to C1, C4/C2/C2 to C2, +/C14 to C21, C1 to C22, +/C15 to C23, R9/+/+1 to C3, C21 to C31, C22 to C32, C23 to C33, C24 to C34, C7/+/+1 to C4, C6/R1/C3 to C5, +/C6/C6 to C6, C8/C5/C5 to C7, C1/+/-1 to C8, C9/+/-1 to C9, +/D1 to D1, +/L1 to L1, +/L2/L2 to L2, +/L3 to L3, Q3/+1/+1 to Q2, Q2 to Q3, +/Q4 to Q4, R1/R1/R1 to R1, R12/-1 to R10, R14/R4/R4 to R11, R2/R5/+1 to R12, R16/+1/R5 to R13, R4/+/-1 to R14, R3/+/+1 to R15, R17/+/+1 to R16, R6/+/+1 to R17, R10 to R18, R12 to R19, D1/R2/R2 to R2, +/R27 to R21, +/R28 to R22, +/R1 to R23, +/R29 to R24, +/R30 to R25, +/R17 to R26, R8/1/+1 to R3, R7/-/-1 to R4, R11/+/+1 to R5, R10/-1 to R6, C6/R3 to R7, -/-/-1 to R8, +/+1 to R9, RV/+1 to RV_Trim1
Connections:
- net GND: now also R19.2, R26.2, RV3.1; no longer RV3.2, RV3.3
- net at C16.2: now also Output1.2 (Pin_2), R19.1; no longer R19.2
- net at C23.2: now also C2.1, C3.1, C4.1, R26.1, R9.2; no longer R26.2
- net at R10.1: now also RV3.2; no longer RV3.1
- no-connect marks 11 -> 12
Other:
- moved on the sheet: R19, R26, RV3

Commit message: Anfang von Bautteilliste
Parts:
- renumbered C16 to C10, J4 to Taster1
Changed lines of the file:
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@@
   (symbol (lib_id "Device:C_Small") (at 241.554 108.966 90) (unit 1)
     (in_bom yes) (on_board yes) (dnp no)
-    (property "Reference" "C16" (at 240.03 112.268 90)
+    (property "Reference" "C10" (at 240.03 112.268 90)
       (effects (font (size 1.27 1.27)))
     )
@@
       (project "KiKAD_Endplatine_V2"
         (path "/06aebb48-3bd9-4517-ad22-b5366be0f5d8"
-          (reference "C16") (unit 1)
+          (reference "C10") (unit 1)
         )
       )
@@
   (symbol (lib_id "Connector:Conn_01x03_Pin") (at 56.388 59.69 0) (unit 1)
     (in_bom yes) (on_board yes) (dnp no)
-    (property "Reference" "J4" (at 57.023 53.086 0)
+    (property "Reference" "Taster1" (at 53.34 55.88 0)
       (effects (font (size 1.27 1.27)))
     )
@@
       (project "KiKAD_Endplatine_V2"
         (path "/06aebb48-3bd9-4517-ad22-b5366be0f5d8"
-          (reference "J4") (unit 1)
-        )
-      )
+          (reference "Taster1") (unit 1)
+        )
+      )

Commit message: Bautteilliste Update
Neue Bautteilliste jtzt in Doku Ordner
KiCad Namensstruktur verändert und jaaa
Parts:
- removed R8, R9: 1000k, Resistor_SMD:R_1206_3216Metric_Pad1.30x1.75mm_HandSolder, symbol Device:R
- removed RV2: 10k, Connector_JST:JST_EH_S2B-EH_1x02_P2.50mm_Horizontal, symbol Device:R_Potentiometer
- C31: value 1p -> 100n
- C32: value 100n -> 10n
- C33: value 10p -> 10u
- R32: value 10k -> 47k
- R33: value 214 -> 220
- R34: value 1k -> 10k
- RV3: value 10k -> 1k
Connections:
- net at R2.2, R4.1: now also RV1.1; no longer RV1.2
- net at R6.2, R7.1: now also C3.2, C5.1
- net at R3.2: now also RV1.2; no longer RV1.3
Other:
- moved on the sheet: R3, RV1
