File: kicad/Finale Platine/KiKAD_Endplatine_V2-backups/KiKAD_Endplatine_V2-2023-09-12_112743/KiKAD_Endplatine_V2.kicad_pcb (KiCad board)
At the start: 2 copper layers, 100 x 80 mm, 70 parts, among them J1 Conn_02x08_Odd_Even, J4 Conn_01x03_Pin, Q1 Q_NPN_ECB, Q2 Q_NPN_ECB, Q3/+1/+1 Q_NPN_ECB, U1 NE555P, U2 TL074

Commit message: aufräumaktion
Parts:
- D2: value C5/D2/D2 -> C5/C5/D2
- R8/R8/+1: renamed from R8/1/+1; value 1000k -> 5k
- renumbered +/C14 to +/+/C14, C1 to +/+/C15, +/C15 to +/+/C16, +/C6/C6 to +/+/C6, +/L1 to +/+/L1, +/L2/L2 to +/+/L2, +/L3 to +/+/L3, +/Q4 to +/+/Q4, +/R1 to +/+/R1, +/R17 to +/+/R17, +/R27 to +/+/R27, +/R28 to +/+/R28, +/R29 to +/+/R29, C6/R3 to +/+/R3, +/R30 to +/+/R30, +/RV1 to +/+/RV1, +/RV3 to +/+/RV3, C1/+/-1 to +/C1/-1, C9/+/-1 to +/C2/-1, Q3/+1/+1 to +/Q3/+1, R16/+1/R5 to +/R16/R5, R17/+/+1 to +/R17/+1, R2/R5/+1 to +/R2/+1, R3/+/+1 to +/R3/+1, R4/+/-1 to +/R4/-1, +/D1 to +/R5/D1, R6/+/+1 to +/R6/+1, C3/C1 to C3/C3/C1, C4/C2/C2 to C4/C4/C2, C6/R1/C3 to C6/C6/C3, C7/+/+1 to C7/C7/+1, C8/C5/C5 to C8/C8/C5, D1/R2/R2 to D1/D1/R2, R10/-1 to R10/10/-1, R11/+/+1 to R11/R11/+1, R12/-1 to R12/R12/-1, R14/R4/R4 to R14/R14/R4, RV/+1 to R5/+/+1, R7/-/-1 to R7/R7/-1, R9/+/+1 to R9/R9/+1, RV1k/-/-1 to RV1k/RV1k/-1
Connections:
- +/+/C14 pad 1: Net-(+/Q4-C) -> Net-(+/+/Q4-E)
- +/+/Q4 pad 1: unconnected-(+/Q4-E-Pad1) -> Net-(+/+/Q4-E)
- +/+/Q4 pad 2: Net-(+/Q4-C) -> unconnected-(+/+/Q4-C-Pad2)
- +/+/R27 pad 2: Net-(+/Q4-C) -> Net-(+/+/Q4-E)
Routing:
- net Net-(+/Q4-C): track 8.14 -> 0.00 mm
- net (no net): track 0.00 -> 8.14 mm
