File: kicad/summierer/summierer/summierer.kicad_sch (KiCad schematic)
At the start: 20 parts, among them J1 IDC_16, J12 OUT1, J2 IN1, J3 IN2, J4 IN3, J5 IN4, J6 IN5, J7 IN6, J8 IN7, J9 IN8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

Commit message: ergänzung summierer
Other:
- note added: "Alle R: 10k Technisch sauberer wäre es die 8 Eingangssignale und das Ausgangssignal über 1µF Kondensatoren ein- bzw. Auszukoppeln. Aus Kostengründen wurde darauf verzichtet Implementierung auf Lochrasterplatine, daher keine PCB-Datei"
- note removed: "Alle R: 10k Technisch sauberer wäre es die 8 Eingangssignale und das Ausgangssignal über 1µF Kondensatoren ein- bzw. Auszukoppeln. Aus Kostengründen wurde darauf verzichtet"
Changed lines of the file:
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@@
     (stroke (width 0) (type default))
   )
-  (text "Alle R: 10k\n\nTechnisch sauberer wäre es die 8 Eingangssignale und das Ausgangssignal über 1µF Kondensatoren ein- bzw. Auszukoppeln.\nAus Kostengründen wurde darauf verzichtet\n"
-    (at 15.24 86.36 0)
+  (text "Alle R: 10k\n\nTechnisch sauberer wäre es die 8 Eingangssignale und das Ausgangssignal über 1µF Kondensatoren ein- bzw. Auszukoppeln.\nAus Kostengründen wurde darauf verzichtet\n\nImplementierung auf Lochrasterplatine, daher keine PCB-Datei\n\n"
+    (at 14.605 95.885 0)
     (effects (font (size 1.27 1.27)) (justify left bottom))
   )
