File: kicad/Klangplatinen/Final_Platine_2/KiKAD_Final_Platine_2_V1.kicad_sch (KiCad schematic)
At the start: 33 parts, among them J1 Conn_02x08_Odd_Even, J4 Conn_01x03_Pin, Q1 Q_NPN_ECB, Q2 Q_NPN_ECB, U1 NE555P, U2 AD8603

Commit message: hää
Parts:
- removed Noise_Input1: Conn_01x02_Pin, Connector_JST:JST_EH_S2B-EH_1x02_P2.50mm_Horizontal, symbol Connector:Conn_01x02_Pin
- added C11, C6: 1u, Capacitor_SMD:C_1206_3216Metric_Pad1.33x1.80mm_HandSolder, symbol Device:C_Small
- added Q3: Q_NPN_ECB, Package_TO_SOT_SMD:SOT-23-3, symbol Device:Q_NPN_ECB
- added R11: 1k, Resistor_SMD:R_1206_3216Metric_Pad1.30x1.75mm_HandSolder, symbol Device:R
- added R5, R6, R9: 100k, Resistor_SMD:R_1206_3216Metric_Pad1.30x1.75mm_HandSolder, symbol Device:R
- added R8: 680, Resistor_SMD:R_1206_3216Metric_Pad1.30x1.75mm_HandSolder, symbol Device:R
- added U3: AD8603, Package_TO_SOT_SMD:TSOT-23-5, symbol Amplifier_Operational:AD8603
Connections:
- net +12V: now also R5.1, U3.5 (V+)
- net -12V: now also U3.2 (V-)
- net GND: now also Q3.3 (B), R11.2, R6.2, R8.1
- net at C1.1: now also D2.2 (A), R4.2
- new net: R8.2, R9.2, U3.4 (-)
- new net: C1.2, C11.2, R11.1
- new net: C6.1, Q3.1 (E), R5.2
- new net: C11.1, R9.1, U3.1
- new net: C6.2, R6.1, U3.3 (+)
- no-connect marks 5 -> 6
Other:
- moved on the sheet: C1
