File: kicad/klangerzeugung/KiKAD_Endplatine_V2.kicad_sch (KiCad schematic)
At the start: 62 parts, among them J1 Conn_02x08_Odd_Even, Q1 Q_NPN_BEC, Q2 Q_NPN_BEC, Q3 Q_NPN_BEC, Q4 Q_NPN_BEC, U1 NE555P, U2 TL074

Commit message: Schaltungsplan Update
Massebezug hergestellt, update zu Footprints
Parts:
- L1, L2, L3: footprint Inductor_THT:L_Radial_D12.0mm_P6.00mm_Murata_1900R -> Inductor_THT:L_Radial_D8.7mm_P5.00mm_Fastron_07HCP
Changed lines of the file:
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@@
       (effects (font (size 1.27 1.27)) (justify left))
     )
-    (property "Footprint" "Inductor_THT:L_Radial_D12.0mm_P6.00mm_Murata_1900R" (at 116.84 105.918 0)
+    (property "Footprint" "Inductor_THT:L_Radial_D8.7mm_P5.00mm_Fastron_07HCP" (at 116.84 105.918 0)
       (effects (font (size 1.27 1.27)) hide)
     )
@@
       (effects (font (size 1.27 1.27)) (justify left))
     )
-    (property "Footprint" "Inductor_THT:L_Radial_D12.0mm_P6.00mm_Murata_1900R" (at 116.84 98.298 0)
+    (property "Footprint" "Inductor_THT:L_Radial_D8.7mm_P5.00mm_Fastron_07HCP" (at 116.84 98.298 0)
       (effects (font (size 1.27 1.27)) hide)
     )
@@
       (effects (font (size 1.27 1.27)) (justify left))
     )
-    (property "Footprint" "Inductor_THT:L_Radial_D12.0mm_P6.00mm_Murata_1900R" (at 116.84 90.678 0)
-      (effects (font (size 1.27 1.27)) hide)
-    )
+    (property "Footprint" "Inductor_THT:L_Radial_D8.7mm_P5.00mm_Fastron_07HCP" (at 116.84 90.678 0)
+      (effects (font (size 1.27 1.27)) hide)
+    )

Commit message: Update 2 zu Platinen
Parts:
- Output1: footprint Connector_JST:JST_EH_S2B-EH_1x02_P2.50mm_Horizontal -> Connector_JST:JST_EH_B2B-EH-A_1x02_P2.50mm_Vertical
Changed lines of the file:
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@@
       (effects (font (size 1.27 1.27)) (justify right))
     )
-    (property "Footprint" "Connector_JST:JST_EH_S2B-EH_1x02_P2.50mm_Horizontal" (at 262.128 111.506 0)
+    (property "Footprint" "Connector_JST:JST_EH_B2B-EH-A_1x02_P2.50mm_Vertical" (at 262.128 111.506 0)
       (effects (font (size 1.27 1.27)) hide)
     )
