File: kicad/klangerzeugung/Platine V4/Platine V4.kicad_pcb (KiCad board)
At the start: 2 copper layers, 100 x 80 mm, 67 parts, among them M1 1M, M2 82n, Q1 Q_NPN_BEC, Q2 Q_NPN_BEC, Q3 Q_NPN_BEC, Q4 Q_NPN_BEC, U1 NE555P, U2 TL074

Commit message: Platinenbeschriftung
Jetzt auch mit einer Platinen Beschriftung:
Platine 4
EDC (EIB DrumComputer)
Other:
- board text added: "Platine V4 EDC"
Changed lines of the file:
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@@
+    (effects (font (size 1.5 1.5) (thickness 0.3) bold) (justify left bottom))
+  )
+  (gr_text "Platine V4\nEDC\n" (at 175.5 113.25) (layer "F.Cu")
     (effects (font (size 1.5 1.5) (thickness 0.3) bold) (justify left bottom))
   )
